File: CAD/pic-writing-board.kicad_sch (KiCad schematic)
At the start: 16 parts

Commit message: make sch
Parts:
- removed IC?: TMUX1309BQBR, TMUX1309BQBR, symbol TMUX1309BQBR:TMUX1309BQBR
- removed U? (x5): TLP172AM, Package_SO:MFSOP6-4_4.4x3.6mm_P1.27mm, symbol Relay_SolidState:TLP175A
- added C? (x2): 0.1u, Capacitor_SMD:C_0603_1608Metric, symbol Device:C_Small
- added C?: 0.1u(1005, Capacitor_SMD:C_0402_1005Metric, symbol Device:C_Small
- added IC?: TMUX1309BQBR, TMUX1309BQBR, symbol TMUX1309BQBR:TMUX1309BQBR
- added JP?: SolderJumper, Jumper:SolderJumper-2_P1.3mm_Open_RoundedPad1.0x1.5mm, symbol Jumper:SolderJumper_2_Open
- added R? (x10): 10k, Resistor_SMD:R_0603_1608Metric, symbol Device:R_Small
- added R? (x3): 390, Resistor_SMD:R_0603_1608Metric, symbol Device:R_Small
- added U? (x4): TLP172AM, Package_SO:SOIC-4_4.55x3.7mm_P2.54mm, symbol Relay_SolidState:TLP175A
Connections:
- net +5V: now also IC?.17 (VDD), U?.3 (PS), U?.3 (PS), C?.1, C?.1, IC?.16 (VDD), R?.1, R?.1, R?.1, U?.4
- net +9V: now also IC?.1 (VCC+), C?.1, R?.1, R?.1, R?.1, R?.1, R?.1
- net Check18: now also IC?.8 (IN+3), R?.2
- net Check20: now also IC?.11 (IN+4), R?.2
- net Check28: now also IC?.6 (IN+2), R?.2
- net Check8: now also IC?.4 (IN+1), R?.2
- net GND: now also IC?.12 (VCC-), IC?.16 (VSS_2), IC?.17 (GND), IC?.29 (EP), IC?.5 (VSS_1), U?.1 (NS), U?.1 (NS), C?.2, C?.2, C?.2, IC?.6 (~{EN}), IC?.8 (GND), R?.1, R?.1, U?.3, U?.6
- net MCLR: now also JP?.1 (A), U?.4, U?.4
- net MCLR8-18: now also U?.6
- net PGC: now also IC?.24 (RB6/ICSPCLK), IC?.3 (DB)
- net PGC18: now also IC?.2 (S2B)
- net PGC8: now also IC?.5 (S1B)
- net PGD: now also IC?.25 (RB7/ICSPDAT), IC?.13 (DA)
- net PGD18: now also IC?.15 (S2A)
- net PGD8-PGC28: now also IC?.14 (S1A), IC?.4 (S3B)
- net VDD18: now also U?.5 (PD), U?.6 (PD)
- net VDD28: now also U?.5 (PD), U?.6 (PD)
- net VDD8-MCLR28: now also U?.6, U?.6
- net VSS18: now also U?.7 (ND), U?.8 (ND)
- net VSS28: now also U?.7 (ND), U?.8 (ND)
- net VSS8-PGD28: now also IC?.11 (S3A), U?.4
- net VSS28_CTL: now reaches U?.2 (NG)
- net VSS28_CTL: now also IC?.11 (RC3), R?.2
- net VDD28_CTL: now reaches U?.4 (PG)
- net VDD28_CTL: now also IC?.12 (RC4), R?.2
- net VSS18_CTL: now reaches U?.2 (NG)
- net VSS18_CTL: now also IC?.21 (RB3), R?.2
- net VDD18_CTL: now reaches U?.4 (PG)
- net VDD18_CTL: now also IC?.22 (RB4), R?.2
- net Check20_DET: now reaches IC?.13 (OUT4)
- net Check20_DET: now also IC?.2 (RA3)
- net Check18_DET: now reaches IC?.14 (OUT3)
- net Check18_DET: now also IC?.1 (RA2)
- net Check28_DET: now reaches IC?.15 (OUT2)
- net Check28_DET: now also IC?.28 (RA1)
- net Check8_DET: now reaches IC?.16 (OUT1)
- net Check8_DET: now also IC?.23 (RB5)
- net Vref: now reaches IC?.2 (IN-1)
- net Vref: now also IC?.5 (IN-2), IC?.7 (IN-3), IC?.9 (IN-4), R?.2, R?.2
- net VDD8_CTL: now reaches IC?.10 (RC2)
- net VDD8_CTL: now also U?.1, U?.3
- net MCLR8-18_CTL: now reaches IC?.13 (RC5)
- net MCLR8-18_CTL: now also R?.1
- net MCLR28_CTL: now reaches IC?.14 (RC6)
- net MCLR28_CTL: now also R?.2
- net at IC?.26 (RE3/~{MCLR}/VPP): now also JP?.2 (B)
- net B: now reaches IC?.8 (RC0)
- net B: now also IC?.9 (A1), U?.3
- net A: now reaches IC?.9 (RC1)
- net A: now also IC?.10 (A0), R?.1
- new net: R?.2, U?.1 (x2)
- new net: R?.1, U?.1, U?.3
- no-connect marks 27 -> 41
Other:
- note added: "Detect to Low"
- note added: "GND"
- note added: "Internal Pullup"
- note added: "MCLR"
- note added: "MCLR-VDD"
- note added: "MCU"
- note added: "MUX"
- note added: "Pin Detect"
- note added: "Power"
- moved on the sheet: C?, IC?, J?, U?

Commit message: import parts
Parts:
- C2, C3: renamed from C?; footprint (none) -> Capacitor_SMD:C_0603_1608Metric
- C4: renamed from C?; value 0.1u(1005 -> 0.1u; footprint Capacitor_SMD:C_0402_1005Metric -> Capacitor_SMD:C_0603_1608Metric
- IC1: renamed from IC?; footprint QFN50P300X300X100-17N -> lib:QFN50P300X300X100-17N
- IC2: renamed from IC?; footprint QFN65P600X600X100-29N-D -> lib:QFN65P600X600X100-29N-D
- IC3: renamed from IC?; footprint TMUX1309BQBR -> lib:TMUX1309BQBR
- J1: renamed from J?; footprint (none) -> Connector_BarrelJack:BarrelJack_Wuerth_6941xx301002
- J2: renamed from J?; footprint Gentiana:ZIF -> lib:ZIF
- J3: renamed from J?; footprint (none) -> lib:6P6C
- U1, U2: renamed from U?; footprint (none) -> Package_SO:SOP-8_3.9x4.9mm_P1.27mm
- U3: renamed from U?; footprint (none) -> Package_TO_SOT_SMD:TO-252-2
- gave numbers to parts that had none: 20

Commit message: adjust port assign
Connections:
- net MCLR: now also U5.6; no longer U5.4
- net VDD8-MCLR28: now also U5.4; no longer U5.6
Changed lines of the file:
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@@
     (effects (font (size 1.27 1.27)) (justify left bottom))
   )
-  (label "VDD8-MCLR28" (at 129.54 142.24 0)
+  (label "VDD8-MCLR28" (at 129.54 147.32 0)
     (effects (font (size 1.27 1.27)) (justify left bottom))
   )
@@
     (effects (font (size 1.27 1.27)) (justify left bottom))
   )
-  (label "MCLR" (at 129.54 147.32 0)
+  (label "MCLR" (at 129.54 142.24 0)
     (effects (font (size 1.27 1.27)) (justify left bottom))
   )

Commit message: make pcb
Connections:
- net A: now also IC2.1 (RA2); no longer IC2.9 (RC1)
- net B: now also IC2.28 (RA1); no longer IC2.8 (RC0)
- net Check18_DET: no longer IC2.1 (RA2)
- net Check20_DET: no longer IC2.2 (RA3)
- net Check28_DET: no longer IC2.28 (RA1)
- net Check8_DET: no longer IC2.23 (RB5)
- net MCLR28_CTL: no longer IC2.14 (RC6)
- net MCLR8-18_CTL: no longer IC2.13 (RC5)
- net VDD18_CTL: no longer IC2.22 (RB4)
- net VDD28_CTL: now also IC2.22 (RB4); no longer IC2.12 (RC4)
- net VDD8_CTL: no longer IC2.10 (RC2)
- net VSS18_CTL: no longer IC2.21 (RB3)
- net VSS28_CTL: now also IC2.23 (RB5); no longer IC2.11 (RC3)
Changed lines of the file:
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@@
+    (stroke (width 0) (type default) (color 0 0 0 0))
+  )
+  (wire (pts (xy 189.23 43.18) (xy 193.04 43.18))
     (stroke (width 0) (type default) (color 0 0 0 0))
   )
@@
     (stroke (width 0) (type default) (color 0 0 0 0))
   )
-  (wire (pts (xy 193.04 43.18) (xy 189.23 43.18))
-    (stroke (width 0) (type default) (color 0 0 0 0))
-  )
   (wire (pts (xy 95.25 87.63) (xy 97.79 87.63))
     (stroke (width 0) (type default) (color 0 0 0 0))
@@
     (stroke (width 0) (type default) (color 0 0 0 0))
   )
-  (wire (pts (xy 171.45 105.41) (xy 168.91 105.41))
-    (stroke (width 0) (type default) (color 0 0 0 0))
-  )
   (wire (pts (xy 115.57 83.82) (xy 127 83.82))
     (stroke (width 0) (type default) (color 0 0 0 0))
@@
     (stroke (width 0) (type default) (color 0 0 0 0))
   )
-  (wire (pts (xy 189.23 107.95) (xy 184.15 107.95))
-    (stroke (width 0) (type default) (color 0 0 0 0))
-  )
   (wire (pts (xy 193.04 34.29) (xy 181.61 34.29))
     (stroke (width 0) (type default) (color 0 0 0 0))
@@
     (stroke (width 0) (type default) (color 0 0 0 0))
   )
+  (wire (pts (xy 186.69 40.64) (xy 193.04 40.64))
+    (stroke (width 0) (type default) (color 0 0 0 0))
+  )
   (wire (pts (xy 172.72 142.24) (xy 173.99 142.24))
     (stroke (width 0) (type default) (color 0 0 0 0))
@@
     (stroke (width 0) (type default) (color 0 0 0 0))
   )
-  (wire (pts (xy 189.23 110.49) (xy 181.61 110.49))
-    (stroke (width 0) (type default) (color 0 0 0 0))
-  )
   (wire (pts (xy 57.15 113.03) (xy 62.23 113.03))
     (stroke (width 0) (type default) (color 0 0 0 0))
@@
     (stroke (width 0) (type default) (color 0 0 0 0))
   )
-  (wire (pts (xy 196.85 72.39) (xy 201.93 72.39))
-    (stroke (width 0) (type default) (color 0 0 0 0))
-  )
   (wire (pts (xy 161.29 82.55) (xy 163.83 82.55))
     (stroke (width 0) (type default) (color 0 0 0 0))
@@
     (stroke (width 0) (type default) (color 0 0 0 0))
   )
-  (wire (pts (xy 193.04 40.64) (xy 186.69 40.64))
-    (stroke (width 0) (type default) (color 0 0 0 0))
-  )
-  (wire (pts (xy 171.45 41.91) (xy 173.99 41.91))
-    (stroke (width 0) (type default) (color 0 0 0 0))
-  )
   (wire (pts (xy 199.39 82.55) (xy 196.85 82.55))
     (stroke (width 0) (type default) (color 0 0 0 0))
@@
     (stroke (width 0) (type default) (color 0 0 0 0))
   )
-  (wire (pts (xy 189.23 105.41) (xy 186.69 105.41))
-    (stroke (width 0) (type default) (color 0 0 0 0))
-  )
   (wire (pts (xy 127 83.82) (xy 127 82.55))
     (stroke (width 0) (type default) (color 0 0 0 0))
   )
-  (wire (pts (xy 173.99 41.91) (xy 173.99 44.45))
+  (wire (pts (xy 173.99 40.64) (xy 173.99 44.45))
     (stroke (width 0) (type default) (color 0 0 0 0))
   )
@@
     (stroke (width 0) (type default) (color 0 0 0 0))
   )
+  (wire (pts (xy 170.18 40.64) (xy 173.99 40.64))
+    (stroke (width 0) (type default) (color 0 0 0 0))
+  )
   (wire (pts (xy 238.76 83.82) (xy 238.76 85.09))
     (stroke (width 0) (type default) (color 0 0 0 0))
@@
     (stroke (width 0) (type default) (color 0 0 0 0))
   )
-  (wire (pts (xy 176.53 110.49) (xy 168.91 110.49))
-    (stroke (width 0) (type default) (color 0 0 0 0))
-  )
   (wire (pts (xy 35.56 144.78) (xy 31.75 144.78))
     (stroke (width 0) (type default) (color 0 0 0 0))
@@
     (stroke (width 0) (type default) (color 0 0 0 0))
   )
-  (wire (pts (xy 168.91 107.95) (xy 173.99 107.95))
-    (stroke (width 0) (type default) (color 0 0 0 0))
-  )
-  (wire (pts (xy 189.23 113.03) (xy 179.07 113.03))
-    (stroke (width 0) (type default) (color 0 0 0 0))
-  )
   (wire (pts (xy 49.53 153.67) (xy 52.07 153.67))
     (stroke (width 0) (type default) (color 0 0 0 0))
@@
     (effects (font (size 1.27 1.27)) (justify right bottom))
   )
-  (label "B" (at 168.91 105.41 180)
+  (label "B" (at 170.18 40.64 180)
     (effects (font (size 1.27 1.27)) (justify right bottom))
   )
@@
     (effects (font (size 1.27 1.27)) (justify left bottom))
   )
-  (label "Check20_DET" (at 163.83 74.93 180)
+  (label "Check20_DET" (at 158.75 74.93 180)
     (effects (font (size 1.27 1.27)) (justify right bottom))
   )
@@
     (effects (font (size 1.27 1.27)) (justify left bottom))
   )
-  (label "Check18_DET" (at 163.83 72.39 180)
+  (label "Check18_DET" (at 158.75 72.39 180)
     (effects (font (size 1.27 1.27)) (justify right bottom))
   )
@@
     (effects (font (size 1.27 1.27)) (justify left bottom))
   )
-  (label "Check8_DET" (at 193.04 40.64 0)
+  (label "Check8_DET" (at 189.23 100.33 0)
     (effects (font (size 1.27 1.27)) (justify left bottom))
   )
@@
     (effects (font (size 1.27 1.27)) (justify right bottom))
   )
-  (label "VDD18_CTL" (at 193.04 43.18 0)
+  (label "VDD18_CTL" (at 189.23 102.87 0)
     (effects (font (size 1.27 1.27)) (justify left bottom))
   )
@@
     (effects (font (size 1.27 1.27)) (justify left bottom))
   )
-  (label "A" (at 168.91 107.95 180)
+  (label "A" (at 163.83 72.39 180)
     (effects (font (size 1.27 1.27)) (justify right bottom))
   )
@@
     (effects (font (size 1.27 1.27)) (justify left bottom))
   )
-  (label "VDD8_CTL" (at 168.91 110.49 180)
+  (label "VDD8_CTL" (at 165.1 110.49 180)
     (effects (font (size 1.27 1.27)) (justify right bottom))
   )
@@
     (effects (font (size 1.27 1.27)) (justify left bottom))
   )
-  (label "VDD28_CTL" (at 189.23 110.49 0)
+  (label "VDD28_CTL" (at 193.04 43.18 0)
     (effects (font (size 1.27 1.27)) (justify left bottom))
   )
@@
     (effects (font (size 1.27 1.27)) (justify right bottom))
   )
-  (label "VSS28_CTL" (at 189.23 113.03 0)
+  (label "VSS28_CTL" (at 193.04 40.64 0)
     (effects (font (size 1.27 1.27)) (justify left bottom))
   )
@@
     (effects (font (size 1.27 1.27)) (justify right bottom))
   )
-  (label "Check28_DET" (at 171.45 41.91 180)
-    (effects (font (size 1.27 1.27)) (justify right bottom))
-  )
+  (label "Check28_DET" (at 165.1 105.41 180)
+    (effects (font (size 1.27 1.27)) (justify right bottom))
+  )

Commit message: adjust sch
Connections:
- net Check18: now also IC1.11 (IN+4), R11.2; no longer IC1.8 (IN+3), R10.2
- net Check18_DET: now also IC1.13 (OUT4), IC2.13 (RC5); no longer IC1.14 (OUT3)
- net Check20: now also IC1.8 (IN+3), R10.2; no longer IC1.11 (IN+4), R11.2
- net Check20_DET: now also IC1.14 (OUT3), IC2.12 (RC4); no longer IC1.13 (OUT4)
- net Check28_DET: now also IC2.10 (RC2)
- net Check8_DET: now also IC2.9 (RC1)
- net MCLR28_CTL: now also IC2.19 (RB1)
- net MCLR8-18_CTL: now also IC2.21 (RB3)
- net VDD18_CTL: now also IC2.3 (RA4)
- net VDD8_CTL: now also IC2.20 (RB2)
- net VSS18_CTL: now also IC2.2 (RA3)
