File: CAD/pic-writing-board.kicad_pcb (KiCad board)
At the start: 2 copper layers, 32 parts, among them IC1 LM2901Q4T, IC2 PIC18F27Q10-I_ML, IC3 TMUX1309BQBR, J1 Barrel_Jack_Switch, J2 ZIF, J3 RJ12, U1 TCP8407, U2 TCP8407, U3 NJM2845, U4 TLP172AM, U5 TLP172AM, U6 TLP172AM, U7 TLP172AM

Commit message: make pcb
Parts:
- added REF**: MountingHole_3.2mm_M3, MountingHole:MountingHole_3.2mm_M3, F.Cu at (97.8, 109.9)
- added REF**: MountingHole_3.2mm_M3, MountingHole:MountingHole_3.2mm_M3, F.Cu at (137.8, 109.9)
- added REF**: MountingHole_3.2mm_M3, MountingHole:MountingHole_3.2mm_M3, F.Cu at (97.8, 51.4)
- added REF**: MountingHole_3.2mm_M3, MountingHole:MountingHole_3.2mm_M3, F.Cu at (137.8, 51.4)
- C1, C2, C3, C4, C5, IC1, IC2, IC3, JP1, R1, R10, R11, R12, R13, R2, R3, R4, R5, R6, R7, R8, R9, U1, U2, U4, U5, U6, U7: moved to B.Cu
- U3: value NJM2845 -> locked; moved to B.Cu
- moved J3 77.2 mm to (100.3, 97.2), turned to -90 degrees
- moved U4 72.3 mm to (115.6, 52.6), turned to -90 degrees
- moved U5 70.9 mm to (109.2, 52.6), turned to -90 degrees
- moved R9 65.9 mm to (106.0, 52.3), turned to -90 degrees
- moved R12 65.5 mm to (118.7, 50.4), turned to 90 degrees
- moved U3 63.9 mm to (101.6, 78.5), turned to 180 degrees
- moved C3 63.3 mm to (105.2, 83.2), turned to 180 degrees
- moved C2 63.2 mm to (104.8, 73.7), turned to 180 degrees
- moved R11 60.5 mm to (108.0, 86.4)
- moved U1 58.8 mm to (123.7, 79.4)
- moved JP1 57.2 mm to (96.5, 92.7)
- moved IC1 56.0 mm to (121.9, 107.3), turned to 180 degrees
- moved R10 54.2 mm to (109.0, 76.2)
- moved R8 52.2 mm to (125.1, 110.7), turned to 90 degrees
- moved R13 51.9 mm to (131.4, 52.3), turned to 90 degrees
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Connections:
- IC1 pad 11: /Check20 -> /Check18
- IC1 pad 13: /Check20_DET -> /Check18_DET
- IC1 pad 14: /Check18_DET -> /Check20_DET
- IC1 pad 8: /Check18 -> /Check20
- IC2 pad 1: /Check18_DET -> /A
- IC2 pad 10: /VDD8_CTL -> /Check28_DET
- IC2 pad 11: /VSS28_CTL -> unconnected-(IC2-Pad11)
- IC2 pad 12: /VDD28_CTL -> /Check20_DET
- IC2 pad 13: /MCLR8-18_CTL -> /Check18_DET
- IC2 pad 14: /MCLR28_CTL -> unconnected-(IC2-Pad14)
- IC2 pad 19: unconnected-(IC2-Pad19) -> /MCLR28_CTL
- IC2 pad 2: /Check20_DET -> /VSS18_CTL
- IC2 pad 20: unconnected-(IC2-Pad20) -> /VDD8_CTL
- IC2 pad 21: /VSS18_CTL -> /MCLR8-18_CTL
- IC2 pad 22: /VDD18_CTL -> /VDD28_CTL
- IC2 pad 23: /Check8_DET -> /VSS28_CTL
- IC2 pad 28: /Check28_DET -> /B
- IC2 pad 3: unconnected-(IC2-Pad3) -> /VDD18_CTL
- IC2 pad 8: /B -> unconnected-(IC2-Pad8)
- IC2 pad 9: /A -> /Check8_DET
- R10 pad 2: /Check18 -> /Check20
- R11 pad 2: /Check20 -> /Check18
- U5 pad 4: /MCLR -> /VDD8-MCLR28
- U5 pad 6: /VDD8-MCLR28 -> /MCLR
Routing:
- net +5V: track 0.00 -> 119.5 mm, vias 0 -> 9
- net +9V: track 0.00 -> 93.3 mm, vias 0 -> 2
- net /MCLR: track 0.00 -> 85.0 mm
- net /B: track 0.00 -> 77.3 mm, vias 0 -> 4
- net /A: track 0.00 -> 71.2 mm, vias 0 -> 4
- net /VSS8-PGD28: track 0.00 -> 67.6 mm, vias 0 -> 2
- net /Check8: track 0.00 -> 59.0 mm, vias 0 -> 1
- net /MCLR28_CTL: track 0.00 -> 57.1 mm, vias 0 -> 2
- net /VDD8_CTL: track 0.00 -> 57.1 mm, vias 0 -> 2
- net /VDD18_CTL: track 0.00 -> 55.4 mm, vias 0 -> 2
- net /VSS18_CTL: track 0.00 -> 53.7 mm, vias 0 -> 2
- net /MCLR8-18_CTL: track 0.00 -> 48.7 mm, vias 0 -> 2
- net /Check20: track 0.00 -> 46.8 mm, vias 0 -> 1
- net /Check18: track 0.00 -> 44.5 mm, vias 0 -> 1
- net /PGD8-PGC28: track 0.00 -> 43.9 mm, vias 0 -> 2
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Other:
- board outline added: 47.6 x 66 mm

Commit message: fill pcb
Parts:
- moved R10 10.2 mm to (108.0, 86.4)
- moved R11 10.2 mm to (109.0, 76.2)
Routing:
- net GND: track 11.4 -> 46.6 mm, vias 2 -> 153
- added copper zone on B.Cu, net GND
- added copper zone on F.Cu, net GND
Other:
- outline, holes or cut-outs redrawn
- rule pad_to_mask_clearance: 0 -> 0.2
